File: CSYNC_ANGLE_CHANGE_MID/RGB_CONN_CHG_MID_98CSYNC_ST.kicad_pcb (KiCad board)
At the start: 2 copper layers, 16 x 16 mm, 5 parts, among them J1 TO_VGA1, J2 TO_VGA1, J3 TO_VGA2, J4 TO_VGA2, J5 C/H

Commit message: update f_silk
added "Licensed under CERN-OHL-W v2"
Other:
- board text added: "Licensed under CERN-OHL-W v2"
