File: DE15_OUT/RGB_CONN_CHG_DE15_CUP_ST.kicad_pcb (KiCad board)
At the start: 2 copper layers, 16 x 16 mm, 3 parts, among them J1 RGB, J2 VGA (C), J3 HV

Commit message: update f_silk
added "Licensed under CERN-OHL-W v2"
Parts:
- J2: value VGA (C) -> VGA
Other:
- board text added: "Licensed under CERN-OHL-W v2"
Changed lines of the file:
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@@
   (general
     (thickness 1.6)
-    (drawings 11)
+    (drawings 12)
     (tracks 23)
     (zones 0)
@@
       (effects (font (size 1 1) (thickness 0.15)))
     )
+    (fp_line (start 1.8 -1.8) (end -1.8 -1.8) (layer F.CrtYd) (width 0.05))
+    (fp_line (start 1.8 6.85) (end 1.8 -1.8) (layer F.CrtYd) (width 0.05))
+    (fp_line (start -1.8 6.85) (end 1.8 6.85) (layer F.CrtYd) (width 0.05))
+    (fp_line (start -1.8 -1.8) (end -1.8 6.85) (layer F.CrtYd) (width 0.05))
+    (fp_line (start -1.33 -1.33) (end 0 -1.33) (layer F.SilkS) (width 0.12))
+    (fp_line (start -1.33 0) (end -1.33 -1.33) (layer F.SilkS) (width 0.12))
+    (fp_line (start -1.33 1.27) (end 1.33 1.27) (layer F.SilkS) (width 0.12))
+    (fp_line (start 1.33 1.27) (end 1.33 6.41) (layer F.SilkS) (width 0.12))
+    (fp_line (start -1.33 1.27) (end -1.33 6.41) (layer F.SilkS) (width 0.12))
+    (fp_line (start -1.33 6.41) (end 1.33 6.41) (layer F.SilkS) (width 0.12))
+    (fp_line (start -1.27 -0.635) (end -0.635 -1.27) (layer F.Fab) (width 0.1))
+    (fp_line (start -1.27 6.35) (end -1.27 -0.635) (layer F.Fab) (width 0.1))
+    (fp_line (start 1.27 6.35) (end -1.27 6.35) (layer F.Fab) (width 0.1))
+    (fp_line (start 1.27 -1.27) (end 1.27 6.35) (layer F.Fab) (width 0.1))
     (fp_line (start -0.635 -1.27) (end 1.27 -1.27) (layer F.Fab) (width 0.1))
-    (fp_line (start 1.27 -1.27) (end 1.27 6.35) (layer F.Fab) (width 0.1))
-    (fp_line (start 1.27 6.35) (end -1.27 6.35) (layer F.Fab) (width 0.1))
-    (fp_line (start -1.27 6.35) (end -1.27 -0.635) (layer F.Fab) (width 0.1))
-    (fp_line (start -1.27 -0.635) (end -0.635 -1.27) (layer F.Fab) (width 0.1))
-    (fp_line (start -1.33 6.41) (end 1.33 6.41) (layer F.SilkS) (width 0.12))
-    (fp_line (start -1.33 1.27) (end -1.33 6.41) (layer F.SilkS) (width 0.12))
-    (fp_line (start 1.33 1.27) (end 1.33 6.41) (layer F.SilkS) (width 0.12))
-    (fp_line (start -1.33 1.27) (end 1.33 1.27) (layer F.SilkS) (width 0.12))
-    (fp_line (start -1.33 0) (end -1.33 -1.33) (layer F.SilkS) (width 0.12))
-    (fp_line (start -1.33 -1.33) (end 0 -1.33) (layer F.SilkS) (width 0.12))
-    (fp_line (start -1.8 -1.8) (end -1.8 6.85) (layer F.CrtYd) (width 0.05))
-    (fp_line (start -1.8 6.85) (end 1.8 6.85) (layer F.CrtYd) (width 0.05))
-    (fp_line (start 1.8 6.85) (end 1.8 -1.8) (layer F.CrtYd) (width 0.05))
-    (fp_line (start 1.8 -1.8) (end -1.8 -1.8) (layer F.CrtYd) (width 0.05))
     (fp_text user %R (at 0 2.54) (layer F.Fab)
       (effects (font (size 1 1) (thickness 0.15)))
@@
       (effects (font (size 1 1) (thickness 0.15)))
     )
+    (fp_line (start 1.8 -1.8) (end -1.8 -1.8) (layer F.CrtYd) (width 0.05))
+    (fp_line (start 1.8 6.85) (end 1.8 -1.8) (layer F.CrtYd) (width 0.05))
+    (fp_line (start -1.8 6.85) (end 1.8 6.85) (layer F.CrtYd) (width 0.05))
+    (fp_line (start -1.8 -1.8) (end -1.8 6.85) (layer F.CrtYd) (width 0.05))
+    (fp_line (start -1.33 -1.33) (end 0 -1.33) (layer F.SilkS) (width 0.12))
+    (fp_line (start -1.33 0) (end -1.33 -1.33) (layer F.SilkS) (width 0.12))
+    (fp_line (start -1.33 1.27) (end 1.33 1.27) (layer F.SilkS) (width 0.12))
+    (fp_line (start 1.33 1.27) (end 1.33 6.41) (layer F.SilkS) (width 0.12))
+    (fp_line (start -1.33 1.27) (end -1.33 6.41) (layer F.SilkS) (width 0.12))
+    (fp_line (start -1.33 6.41) (end 1.33 6.41) (layer F.SilkS) (width 0.12))
+    (fp_line (start -1.27 -0.635) (end -0.635 -1.27) (layer F.Fab) (width 0.1))
+    (fp_line (start -1.27 6.35) (end -1.27 -0.635) (layer F.Fab) (width 0.1))
+    (fp_line (start 1.27 6.35) (end -1.27 6.35) (layer F.Fab) (width 0.1))
+    (fp_line (start 1.27 -1.27) (end 1.27 6.35) (layer F.Fab) (width 0.1))
     (fp_line (start -0.635 -1.27) (end 1.27 -1.27) (layer F.Fab) (width 0.1))
-    (fp_line (start 1.27 -1.27) (end 1.27 6.35) (layer F.Fab) (width 0.1))
-    (fp_line (start 1.27 6.35) (end -1.27 6.35) (layer F.Fab) (width 0.1))
-    (fp_line (start -1.27 6.35) (end -1.27 -0.635) (layer F.Fab) (width 0.1))
-    (fp_line (start -1.27 -0.635) (end -0.635 -1.27) (layer F.Fab) (width 0.1))
-    (fp_line (start -1.33 6.41) (end 1.33 6.41) (layer F.SilkS) (width 0.12))
-    (fp_line (start -1.33 1.27) (end -1.33 6.41) (layer F.SilkS) (width 0.12))
-    (fp_line (start 1.33 1.27) (end 1.33 6.41) (layer F.SilkS) (width 0.12))
-    (fp_line (start -1.33 1.27) (end 1.33 1.27) (layer F.SilkS) (width 0.12))
-    (fp_line (start -1.33 0) (end -1.33 -1.33) (layer F.SilkS) (width 0.12))
-    (fp_line (start -1.33 -1.33) (end 0 -1.33) (layer F.SilkS) (width 0.12))
-    (fp_line (start -1.8 -1.8) (end -1.8 6.85) (layer F.CrtYd) (width 0.05))
-    (fp_line (start -1.8 6.85) (end 1.8 6.85) (layer F.CrtYd) (width 0.05))
-    (fp_line (start 1.8 6.85) (end 1.8 -1.8) (layer F.CrtYd) (width 0.05))
-    (fp_line (start 1.8 -1.8) (end -1.8 -1.8) (layer F.CrtYd) (width 0.05))
     (fp_text user %R (at 0 2.54) (layer F.Fab)
       (effects (font (size 1 1) (thickness 0.15)))
@@
       (effects (font (size 1.524 1.524) (thickness 0.3048)))
     )
-    (fp_text value "VGA (C)" (at -6.9 -13.3 -90) (layer B.SilkS)
+    (fp_text value VGA (at -7 -12.4 -90) (layer B.SilkS)
       (effects (font (size 1.524 1.524) (thickness 0.3048)) (justify mirror))
     )
+    (fp_line (start 15.5 -5.9) (end -15.488 -5.9) (layer F.SilkS) (width 0.381))
+    (fp_line (start -9.017 -15.112) (end -9.017 -5.9) (layer F.SilkS) (width 0.381))
+    (fp_line (start -15.5 -5.9) (end -15.494 -15.112) (layer F.SilkS) (width 0.381))
+    (fp_line (start 15.494 -15.112) (end 15.5 -5.9) (layer F.SilkS) (width 0.381))
+    (fp_line (start 15.494 -15.112) (end -15.494 -15.112) (layer F.SilkS) (width 0.381))
     (fp_line (start 9.017 -6) (end 9.017 -15.112) (layer F.SilkS) (width 0.381))
-    (fp_line (start 15.494 -15.112) (end -15.494 -15.112) (layer F.SilkS) (width 0.381))
-    (fp_line (start 15.494 -15.112) (end 15.5 -5.9) (layer F.SilkS) (width 0.381))
-    (fp_line (start -15.5 -5.9) (end -15.494 -15.112) (layer F.SilkS) (width 0.381))
-    (fp_line (start -9.017 -15.112) (end -9.017 -5.9) (layer F.SilkS) (width 0.381))
-    (fp_line (start 15.5 -5.9) (end -15.488 -5.9) (layer F.SilkS) (width 0.381))
     (pad 3 thru_hole oval (at -0.2667 -13.112) (size 1.6 2.6) (drill oval 1.4 2.2) (layers *.Cu *.Mask)
       (net 1 B))
@@
     )
   )
+  (gr_text "Licensed under\nCERN-OHL-W v2" (at 128 90.3 90) (layer B.SilkS)
+    (effects (font (size 0.5 0.5) (thickness 0.1)) (justify mirror))
+  )
   (gr_text Rev2 (at 141.8 90.8 90) (layer B.SilkS)
