File: DIN6_X1_IN/RGB_CONN_CHG_DIN6_ST.kicad_pcb (KiCad board)
At the start: 2 copper layers, 16 x 16 mm, 9 parts, among them J1 X1, J2 TO_VGA1, J3 TO_VGA2

Commit message: update f_silk
added "Licensed under CERN-OHL-W v2"
Other:
- board text added: "Licensed under CERN-OHL-W v2"
