File: DE9_FM77_IN/RGB_CONN_CHG_DE9_FM77_ST.kicad_pcb (KiCad board)
At the start: 2 copper layers, 16 x 16 mm, 3 parts, among them J1 FM77, J2 RGB, J3 HV

Commit message: Add files via upload
Other:
- board text added: "Licensed under CERN-OHL-W v2"
Changed lines of the file:
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@@
   (general
     (thickness 1.6)
-    (drawings 16)
+    (drawings 17)
     (tracks 36)
     (zones 0)
@@
       (effects (font (size 1 1) (thickness 0.15)))
     )
+    (fp_line (start -0.635 -1.27) (end 1.27 -1.27) (layer F.Fab) (width 0.1))
+    (fp_line (start 1.27 -1.27) (end 1.27 11.43) (layer F.Fab) (width 0.1))
+    (fp_line (start 1.27 11.43) (end -1.27 11.43) (layer F.Fab) (width 0.1))
+    (fp_line (start -1.27 11.43) (end -1.27 -0.635) (layer F.Fab) (width 0.1))
+    (fp_line (start -1.27 -0.635) (end -0.635 -1.27) (layer F.Fab) (width 0.1))
+    (fp_line (start -1.33 11.49) (end 1.33 11.49) (layer F.SilkS) (width 0.12))
+    (fp_line (start -1.33 1.27) (end -1.33 11.49) (layer F.SilkS) (width 0.12))
+    (fp_line (start 1.33 1.27) (end 1.33 11.49) (layer F.SilkS) (width 0.12))
+    (fp_line (start -1.33 1.27) (end 1.33 1.27) (layer F.SilkS) (width 0.12))
+    (fp_line (start -1.33 0) (end -1.33 -1.33) (layer F.SilkS) (width 0.12))
+    (fp_line (start -1.33 -1.33) (end 0 -1.33) (layer F.SilkS) (width 0.12))
+    (fp_line (start -1.8 -1.8) (end -1.8 11.95) (layer F.CrtYd) (width 0.05))
+    (fp_line (start -1.8 11.95) (end 1.8 11.95) (layer F.CrtYd) (width 0.05))
+    (fp_line (start 1.8 11.95) (end 1.8 -1.8) (layer F.CrtYd) (width 0.05))
     (fp_line (start 1.8 -1.8) (end -1.8 -1.8) (layer F.CrtYd) (width 0.05))
-    (fp_line (start 1.8 11.95) (end 1.8 -1.8) (layer F.CrtYd) (width 0.05))
-    (fp_line (start -1.8 11.95) (end 1.8 11.95) (layer F.CrtYd) (width 0.05))
-    (fp_line (start -1.8 -1.8) (end -1.8 11.95) (layer F.CrtYd) (width 0.05))
-    (fp_line (start -1.33 -1.33) (end 0 -1.33) (layer F.SilkS) (width 0.12))
-    (fp_line (start -1.33 0) (end -1.33 -1.33) (layer F.SilkS) (width 0.12))
-    (fp_line (start -1.33 1.27) (end 1.33 1.27) (layer F.SilkS) (width 0.12))
-    (fp_line (start 1.33 1.27) (end 1.33 11.49) (layer F.SilkS) (width 0.12))
-    (fp_line (start -1.33 1.27) (end -1.33 11.49) (layer F.SilkS) (width 0.12))
-    (fp_line (start -1.33 11.49) (end 1.33 11.49) (layer F.SilkS) (width 0.12))
-    (fp_line (start -1.27 -0.635) (end -0.635 -1.27) (layer F.Fab) (width 0.1))
-    (fp_line (start -1.27 11.43) (end -1.27 -0.635) (layer F.Fab) (width 0.1))
-    (fp_line (start 1.27 11.43) (end -1.27 11.43) (layer F.Fab) (width 0.1))
-    (fp_line (start 1.27 -1.27) (end 1.27 11.43) (layer F.Fab) (width 0.1))
-    (fp_line (start -0.635 -1.27) (end 1.27 -1.27) (layer F.Fab) (width 0.1))
     (fp_text user %R (at 0 5.08) (layer F.Fab)
       (effects (font (size 1 1) (thickness 0.15)))
@@
       (effects (font (size 1 1) (thickness 0.15)))
     )
+    (fp_line (start -0.635 -1.27) (end 1.27 -1.27) (layer F.Fab) (width 0.1))
+    (fp_line (start 1.27 -1.27) (end 1.27 6.35) (layer F.Fab) (width 0.1))
+    (fp_line (start 1.27 6.35) (end -1.27 6.35) (layer F.Fab) (width 0.1))
+    (fp_line (start -1.27 6.35) (end -1.27 -0.635) (layer F.Fab) (width 0.1))
+    (fp_line (start -1.27 -0.635) (end -0.635 -1.27) (layer F.Fab) (width 0.1))
+    (fp_line (start -1.33 6.41) (end 1.33 6.41) (layer F.SilkS) (width 0.12))
+    (fp_line (start -1.33 1.27) (end -1.33 6.41) (layer F.SilkS) (width 0.12))
+    (fp_line (start 1.33 1.27) (end 1.33 6.41) (layer F.SilkS) (width 0.12))
+    (fp_line (start -1.33 1.27) (end 1.33 1.27) (layer F.SilkS) (width 0.12))
+    (fp_line (start -1.33 0) (end -1.33 -1.33) (layer F.SilkS) (width 0.12))
+    (fp_line (start -1.33 -1.33) (end 0 -1.33) (layer F.SilkS) (width 0.12))
+    (fp_line (start -1.8 -1.8) (end -1.8 6.85) (layer F.CrtYd) (width 0.05))
+    (fp_line (start -1.8 6.85) (end 1.8 6.85) (layer F.CrtYd) (width 0.05))
+    (fp_line (start 1.8 6.85) (end 1.8 -1.8) (layer F.CrtYd) (width 0.05))
     (fp_line (start 1.8 -1.8) (end -1.8 -1.8) (layer F.CrtYd) (width 0.05))
-    (fp_line (start 1.8 6.85) (end 1.8 -1.8) (layer F.CrtYd) (width 0.05))
-    (fp_line (start -1.8 6.85) (end 1.8 6.85) (layer F.CrtYd) (width 0.05))
-    (fp_line (start -1.8 -1.8) (end -1.8 6.85) (layer F.CrtYd) (width 0.05))
-    (fp_line (start -1.33 -1.33) (end 0 -1.33) (layer F.SilkS) (width 0.12))
-    (fp_line (start -1.33 0) (end -1.33 -1.33) (layer F.SilkS) (width 0.12))
-    (fp_line (start -1.33 1.27) (end 1.33 1.27) (layer F.SilkS) (width 0.12))
-    (fp_line (start 1.33 1.27) (end 1.33 6.41) (layer F.SilkS) (width 0.12))
-    (fp_line (start -1.33 1.27) (end -1.33 6.41) (layer F.SilkS) (width 0.12))
-    (fp_line (start -1.33 6.41) (end 1.33 6.41) (layer F.SilkS) (width 0.12))
-    (fp_line (start -1.27 -0.635) (end -0.635 -1.27) (layer F.Fab) (width 0.1))
-    (fp_line (start -1.27 6.35) (end -1.27 -0.635) (layer F.Fab) (width 0.1))
-    (fp_line (start 1.27 6.35) (end -1.27 6.35) (layer F.Fab) (width 0.1))
-    (fp_line (start 1.27 -1.27) (end 1.27 6.35) (layer F.Fab) (width 0.1))
-    (fp_line (start -0.635 -1.27) (end 1.27 -1.27) (layer F.Fab) (width 0.1))
     (fp_text user %R (at 0 2.54) (layer F.Fab)
       (effects (font (size 1 1) (thickness 0.15)))
@@
       (effects (font (size 1 1) (thickness 0.15)))
     )
+    (fp_line (start -8.885 4.83) (end 19.965 4.83) (layer B.Fab) (width 0.1))
+    (fp_line (start 20.965 3.83) (end 20.965 -6.67) (layer B.Fab) (width 0.1))
+    (fp_line (start 19.965 -7.67) (end -8.885 -7.67) (layer B.Fab) (width 0.1))
+    (fp_line (start -9.885 -6.67) (end -9.885 3.83) (layer B.Fab) (width 0.1))
+    (fp_line (start -8.885 4.89) (end 19.965 4.89) (layer B.SilkS) (width 0.12))
+    (fp_line (start 21.025 3.83) (end 21.025 -6.67) (layer B.SilkS) (width 0.12))
+    (fp_line (start 19.965 -7.73) (end -8.885 -7.73) (layer B.SilkS) (width 0.12))
+    (fp_line (start -9.945 -6.67) (end -9.945 3.83) (layer B.SilkS) (width 0.12))
+    (fp_line (start -0.25 5.784338) (end 0.25 5.784338) (layer B.SilkS) (width 0.12))
+    (fp_line (start 0.25 5.784338) (end 0 5.351325) (layer B.SilkS) (width 0.12))
+    (fp_line (start 0 5.351325) (end -0.25 5.784338) (layer B.SilkS) (width 0.12))
+    (fp_line (start -0.703194 2.73) (end 11.783194 2.73) (layer B.Fab) (width 0.1))
+    (fp_line (start 0.196073 -5.57) (end 10.883927 -5.57) (layer B.Fab) (width 0.1))
+    (fp_line (start 13.358887 0.852163) (end 12.459619 -4.247837) (layer B.Fab) (width 0.1))
+    (fp_line (start -2.278887 0.852163) (end -1.379619 -4.247837) (layer B.Fab) (width 0.1))
+    (fp_line (start -0.691689 2.79) (end 11.771689 2.79) (layer B.SilkS) (width 0.12))
+    (fp_line (start 0.207579 -5.63) (end 10.872421 -5.63) (layer B.SilkS) (width 0.12))
+    (fp_line (start 13.40647 0.841744) (end 12.507202 -4.258256) (layer B.SilkS) (width 0.12))
+    (fp_line (start -2.32647 0.841744) (end -1.427202 -4.258256) (layer B.SilkS) (width 0.12))
+    (fp_line (start -10.4 5.35) (end -10.4 -8.2) (layer B.CrtYd) (width 0.05))
+    (fp_line (start -10.4 -8.2) (end 21.5 -8.2) (layer B.CrtYd) (width 0.05))
+    (fp_line (start 21.5 -8.2) (end 21.5 5.35) (layer B.CrtYd) (width 0.05))
     (fp_line (start 21.5 5.35) (end -10.4 5.35) (layer B.CrtYd) (width 0.05))
-    (fp_line (start 21.5 -8.2) (end 21.5 5.35) (layer B.CrtYd) (width 0.05))
-    (fp_line (start -10.4 -8.2) (end 21.5 -8.2) (layer B.CrtYd) (width 0.05))
-    (fp_line (start -10.4 5.35) (end -10.4 -8.2) (layer B.CrtYd) (width 0.05))
-    (fp_line (start -2.32647 0.841744) (end -1.427202 -4.258256) (layer B.SilkS) (width 0.12))
-    (fp_line (start 13.40647 0.841744) (end 12.507202 -4.258256) (layer B.SilkS) (width 0.12))
-    (fp_line (start 0.207579 -5.63) (end 10.872421 -5.63) (layer B.SilkS) (width 0.12))
-    (fp_line (start -0.691689 2.79) (end 11.771689 2.79) (layer B.SilkS) (width 0.12))
-    (fp_line (start -2.278887 0.852163) (end -1.379619 -4.247837) (layer B.Fab) (width 0.1))
-    (fp_line (start 13.358887 0.852163) (end 12.459619 -4.247837) (layer B.Fab) (width 0.1))
-    (fp_line (start 0.196073 -5.57) (end 10.883927 -5.57) (layer B.Fab) (width 0.1))
-    (fp_line (start -0.703194 2.73) (end 11.783194 2.73) (layer B.Fab) (width 0.1))
-    (fp_line (start 0 5.351325) (end -0.25 5.784338) (layer B.SilkS) (width 0.12))
-    (fp_line (start 0.25 5.784338) (end 0 5.351325) (layer B.SilkS) (width 0.12))
-    (fp_line (start -0.25 5.784338) (end 0.25 5.784338) (layer B.SilkS) (width 0.12))
-    (fp_line (start -9.945 -6.67) (end -9.945 3.83) (layer B.SilkS) (width 0.12))
-    (fp_line (start 19.965 -7.73) (end -8.885 -7.73) (layer B.SilkS) (width 0.12))
-    (fp_line (start 21.025 3.83) (end 21.025 -6.67) (layer B.SilkS) (width 0.12))
-    (fp_line (start -8.885 4.89) (end 19.965 4.89) (layer B.SilkS) (width 0.12))
-    (fp_line (start -9.885 -6.67) (end -9.885 3.83) (layer B.Fab) (width 0.1))
-    (fp_line (start 19.965 -7.67) (end -8.885 -7.67) (layer B.Fab) (width 0.1))
-    (fp_line (start 20.965 3.83) (end 20.965 -6.67) (layer B.Fab) (width 0.1))
-    (fp_line (start -8.885 4.83) (end 19.965 4.83) (layer B.Fab) (width 0.1))
     (fp_text user %R (at 5.54 -1.42) (layer B.Fab)
       (effects (font (size 1 1) (thickness 0.15)) (justify mirror))
@@
     )
   )
+  (gr_text "Licensed under CERN-OHL-W v2" (at 134.9 81.3) (layer B.SilkS)
+    (effects (font (size 0.5 0.5) (thickness 0.1)) (justify mirror))
+  )
   (gr_text I (at 129.9 81.8) (layer F.SilkS)
